File: schematic/8085-explorer.kicad_pcb (KiCad board)
At the start: 2 copper layers, 120 x 80 mm, 51 parts, among them J1 DE9_Pins_MountingHoles, J2 DC-005 Power Jack, J4 Conn_01x02_Pin, J5 Conn_01x02_Pin, J6 Conn_02x05_Odd_Even, U1 8085, U2 74LS573, U3 28C256, U4 HM62256BLP, U5 74LS14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

Commit message: PCB updated
Parts:
- moved C11 1.52 mm to (64.1, 52.1)
- moved C14 1.52 mm to (69.9, 52.1)
Routing:
- net +5V: track 336.9 -> 342.1 mm
- net UART_RX: track 129.6 -> 134.6 mm
- net Net-(U8-VS+): track 14.3 -> 15.9 mm
Other:
- board text added: "ON↓/OFF↑"
- board text added: "RS-232/SERIAL"
- board text removed: "ON/OFF"
- board text removed: "RS232/SERIAL"
Changed lines of the file:
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@@
 	(footprint "Capacitor_THT:CP_Radial_D4.0mm_P2.00mm"
 		(layer "F.Cu")
-		(at 69.8934 53.594)
+		(at 69.8934 52.07)
 		(descr "CP, Radial series, Radial, pin pitch=2.00mm, diameter=4mm, height=7mm, Electrolytic Capacitor")
 		(tags "CP Radial series Radial pin pitch 2.00mm diameter 4mm height 7mm Electrolytic Capacitor")
@@
 	(footprint "Capacitor_THT:CP_Radial_D4.0mm_P2.00mm"
 		(layer "F.Cu")
-		(at 64.0514 53.594)
+		(at 64.0514 52.07)
 		(descr "CP, Radial series, Radial, pin pitch=2.00mm, diameter=4mm, height=7mm, Electrolytic Capacitor")
 		(tags "CP Radial series Radial pin pitch 2.00mm diameter 4mm height 7mm Electrolytic Capacitor")
@@
 		)
 	)
-	(gr_text "ON/OFF"
-		(at 4.572 65.572 0)
+	(gr_text "ON↓/OFF↑"
+		(at 3.556 65.572 0)
 		(layer "F.SilkS")
 		(effects
@@
 	)
 	(gr_text "NETRONICS EXPLORER/85 SINGLE BOARD COMPUTER V1.0"
-		(at 65.1 79.6 0)
+		(at 64.77 79.6 0)
 		(layer "F.SilkS")
 		(effects
@@
 		)
 	)
-	(gr_text "RS232/SERIAL"
-		(at 28.956 75.946 90)
+	(gr_text "RS-232/SERIAL"
+		(at 28.956 77.216 90)
 		(layer "F.SilkS")
 		(effects
@@
 	)
 	(gr_text "2026 B. MARKUS"
-		(at 119.634 68.58 90)
+		(at 119.634 68.326 90)
 		(layer "F.SilkS")
 		(effects
@@
 	)
 	(segment
-		(start 64.774 9.398)
-		(end 59.734 9.398)
+		(start 55.88 54.904)
+		(end 62.7414 54.904)
 		(width 0.2)
 		(layer "F.Cu")
@@
 	)
 	(segment
-		(start 106.421 69.088)
-		(end 105.151 70.358)
+		(start 71.8934 53.594)
+		(end 71.8934 52.07)
 		(width 0.2)
 		(layer "F.Cu")
@@
 	)
 	(segment
-		(start 72.2662 53.9668)
+		(start 71.8934 54.3396)
 		(end 66.548 59.685)
 		(width 0.2)
@@
 	)
 	(segment
-		(start 91.484 58.853)
-		(end 91.484 55.118)
+		(start 64.774 9.398)
+		(end 59.734 9.398)
 		(width 0.2)
 		(layer "F.Cu")
@@
 	)
 	(segment
-		(start 83.3677 55.9667)
-		(end 74.2661 55.9667)
+		(start 106.421 69.088)
+		(end 105.151 70.358)
+		(width 0.2)
+		(layer "F.Cu")
+		(net 1)
+	)
+	(segment
+		(start 91.484 58.853)
+		(end 91.484 55.118)
 		(width 0.2)
 		(layer "F.Cu")
@@
 	)
 	(segment
-		(start 62.7414 54.904)
-		(end 64.0514 53.594)
-		(width 0.2)
-		(layer "F.Cu")
-		(net 1)
-	)
-	(segment
 		(start 38.144 4.318)
 		(end 42.0362 8.2102)
@@
 	)
 	(segment
-		(start 74.2661 55.9667)
-		(end 72.2662 53.9668)
+		(start 90.139 62.738)
+		(end 83.3677 55.9667)
 		(width 0.2)
 		(layer "F.Cu")
@@
 	)
 	(segment
+		(start 71.8934 54.3674)
+		(end 71.8934 53.594)
+		(width 0.2)
+		(layer "F.Cu")
+		(net 1)
+	)
+	(segment
 		(start 91.479 9.398)
 		(end 91.479 4.318)
@@
 	)
 	(segment
+		(start 71.8934 53.594)
+		(end 71.8934 54.3396)
+		(width 0.2)
+		(layer "F.Cu")
+		(net 1)
+	)
+	(segment
+		(start 83.3677 55.9667)
+		(end 73.4927 55.9667)
+		(width 0.2)
+		(layer "F.Cu")
+		(net 1)
+	)
+	(segment
 		(start 97.759 65.278)
 		(end 90.139 65.278)
@@
 	)
 	(segment
-		(start 55.88 54.904)
-		(end 62.7414 54.904)
+		(start 73.4927 55.9667)
+		(end 71.8934 54.3674)
 		(width 0.2)
 		(layer "F.Cu")
@@
 	)
 	(segment
-		(start 90.139 62.738)
-		(end 83.3677 55.9667)
-		(width 0.2)
-		(layer "F.Cu")
-		(net 1)
-	)
-	(segment
-		(start 72.2662 53.9668)
-		(end 71.8934 53.594)
+		(start 62.7414 54.904)
+		(end 64.0514 53.594)
 		(width 0.2)
 		(layer "F.Cu")
@@
 	)
 	(segment
+		(start 64.0514 53.594)
+		(end 64.0514 52.07)
+		(width 0.2)
+		(layer "F.Cu")
+		(net 1)
+	)
+	(segment
 		(start 21.376 4.376)
 		(end 26.398 9.398)
@@
 	)
 	(segment
+		(start 64.0514 57.1884)
+		(end 64.0514 52.07)
+		(width 0.2)
+		(layer "B.Cu")
+		(net 1)
+	)
+	(segment
 		(start 52.578 50.038)
 		(end 45.72 43.18)
@@
 	)
 	(segment
-		(start 64.0514 57.1884)
-		(end 64.0514 53.594)
+		(start 66.548 59.685)
+		(end 64.0514 57.1884)
 		(width 0.2)
 		(layer "B.Cu")
@@
 	)
 	(segment
-		(start 66.548 59.685)
-		(end 64.0514 57.1884)
-		(width 0.2)
-		(layer "B.Cu")
-		(net 1)
-	)
-	(segment
 		(start 38.144 4.318)
 		(end 33.064 9.398)
@@
 	)
 	(segment
-		(start 70.2418 53.9424)
-		(end 69.8934 53.594)
+		(start 69.088 67.305)
+		(end 70.2418 66.1512)
 		(width 0.2)
 		(layer "B.Cu")
@@
 	)
 	(segment
-		(start 69.088 67.305)
-		(end 70.2418 66.1512)
+		(start 70.2418 53.9424)
+		(end 69.8934 53.594)
+		(width 0.2)
+		(layer "B.Cu")
+		(net 10)
+	)
+	(segment
+		(start 69.8934 53.594)
+		(end 69.8934 52.07)
 		(width 0.2)
 		(layer "B.Cu")
@@
 	)
 	(segment
-		(start 68.55 52.676)
-		(end 65.2133 56.0127)
+		(start 16.1097 53.7383)
+		(end 52.5548 53.7383)
 		(width 0.2)
 		(layer "F.Cu")
@@
 	)
 	(segment
-		(start 14.5132 21.5548)
-		(end 16.51 19.558)
+		(start 52.5548 53.7383)
+		(end 54.8292 56.0127)
 		(width 0.2)
 		(layer "F.Cu")
@@
 	)
 	(segment
-		(start 65.2133 56.0127)
-		(end 54.8292 56.0127)
+		(start 14.5132 52.1418)
+		(end 16.1097 53.7383)
 		(width 0.2)
 		(layer "F.Cu")
@@
 	)
 	(segment
-		(start 79.3497 53.34)
-		(end 78.74 53.34)
+		(start 68.58 50.038)
+		(end 74.0323 50.038)
 		(width 0.2)
 		(layer "F.Cu")
@@
 	)
 	(segment
-		(start 78.74 53.34)
-		(end 77.3343 53.34)
+		(start 16.51 19.558)
+		(end 14.5132 21.5548)
 		(width 0.2)
 		(layer "F.Cu")
@@
 	)
 	(segment
-		(start 80.7554 54.7457)
-		(end 79.3497 53.34)
+		(start 68.072 50.546)
+		(end 68.58 50.038)
 		(width 0.2)
 		(layer "F.Cu")
@@
 	)
 	(segment
-		(start 52.5548 53.7383)
-		(end 16.1097 53.7383)
+		(start 68.072 55.372)
+		(end 68.072 50.546)
 		(width 0.2)
 		(layer "F.Cu")
@@
 	)
 	(segment
-		(start 82.7228 54.7457)
-		(end 80.7554 54.7457)
+		(start 79.3497 53.34)
+		(end 78.74 53.34)
 		(width 0.2)
 		(layer "F.Cu")
@@
 	)
 	(segment
-		(start 14.5132 52.1418)
-		(end 14.5132 21.5548)
+		(start 80.7554 54.7457)
+		(end 79.3497 53.34)
 		(width 0.2)
 		(layer "F.Cu")
@@
 	)
 	(segment
-		(start 77.3343 53.34)
-		(end 76.6703 52.676)
+		(start 82.7228 54.7457)
+		(end 80.7554 54.7457)
 		(width 0.2)
 		(layer "F.Cu")
@@
 	)
 	(segment
-		(start 76.6703 52.676)
-		(end 68.55 52.676)
+		(start 74.0323 50.038)
+		(end 77.3343 53.34)
 		(width 0.2)
 		(layer "F.Cu")
@@
 	)
 	(segment
-		(start 16.1097 53.7383)
+		(start 67.4313 56.0127)
+		(end 68.072 55.372)
+		(width 0.2)
+		(layer "F.Cu")
+		(net 21)
+	)
+	(segment
+		(start 14.5132 21.5548)
 		(end 14.5132 52.1418)
 		(width 0.2)
@@
 	(segment
 		(start 54.8292 56.0127)
-		(end 52.5548 53.7383)
+		(end 67.4313 56.0127)
+		(width 0.2)
+		(layer "F.Cu")
+		(net 21)
+	)
+	(segment
+		(start 77.3343 53.34)
+		(end 78.74 53.34)
 		(width 0.2)
 		(layer "F.Cu")

Commit message: PCB updated
Parts:
- moved D4 1.53 mm to (107.7, 7.87)
Routing:
- net Net-(U1-~{RESET_IN}): track 122.6 -> 126.0 mm
- net IO_~{M}: track 184.1 -> 186.3 mm
- net Net-(D4-A): track 9.58 -> 8.94 mm
Changed lines of the file:
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@@
 	(footprint "StockLib:LED_D5.0mm_RED"
 		(layer "F.Cu")
-		(at 106.167 7.874)
+		(at 107.696 7.874)
 		(descr "LED, diameter 5.0mm, 2 pins, http://cdn-reichelt.de/documents/datenblatt/A500/LL-504BC2E-009.pdf")
 		(tags "LED diameter 5.0mm 2 pins")
@@
 	)
 	(gr_text "POWER"
-		(at 104.394 10.414 90)
+		(at 105.918 10.414 90)
 		(layer "F.SilkS")
 		(effects
@@
 	)
 	(segment
-		(start 108.707 8.7993)
-		(end 108.707 7.874)
+		(start 114.046 15.24)
+		(end 114.046 14.1383)
 		(width 0.2)
 		(layer "B.Cu")
@@
 	)
 	(segment
-		(start 114.046 15.24)
-		(end 114.046 14.1383)
+		(start 110.236 10.3283)
+		(end 110.236 7.874)
 		(width 0.2)
 		(layer "B.Cu")
@@
 	(segment
 		(start 114.046 14.1383)
-		(end 108.707 8.7993)
+		(end 110.236 10.3283)
 		(width 0.2)
 		(layer "B.Cu")
@@
 	)
 	(segment
-		(start 110.8232 34.4338)
-		(end 114.8901 34.4338)
+		(start 21.7996 2.3265)
+		(end 20.2232 3.9029)
 		(width 0.2)
 		(layer "F.Cu")
@@
 	)
 	(segment
-		(start 97.759 47.498)
-		(end 110.8232 34.4338)
+		(start 116.2647 9.8387)
+		(end 108.7525 2.3265)
 		(width 0.2)
 		(layer "F.Cu")
@@
 	)
 	(segment
-		(start 116.2647 13.7127)
-		(end 104.8785 2.3265)
+		(start 114.8901 34.4338)
+		(end 116.2647 33.0592)
 		(width 0.2)
 		(layer "F.Cu")
@@
 	)
 	(segment
-		(start 104.8785 2.3265)
-		(end 21.7996 2.3265)
+		(start 20.2232 13.1112)
+		(end 31.75 24.638)
 		(width 0.2)
 		(layer "F.Cu")
@@
 	)
 	(segment
-		(start 20.2232 13.1112)
-		(end 31.75 24.638)
+		(start 20.2232 3.9029)
+		(end 20.2232 13.1112)
 		(width 0.2)
 		(layer "F.Cu")
@@
 	)
 	(segment
-		(start 21.7996 2.3265)
-		(end 20.2232 3.9029)
+		(start 97.759 47.498)
+		(end 110.8232 34.4338)
 		(width 0.2)
 		(layer "F.Cu")
@@
 	)
 	(segment
-		(start 20.2232 3.9029)
-		(end 20.2232 13.1112)
+		(start 108.7525 2.3265)
+		(end 21.7996 2.3265)
 		(width 0.2)
 		(layer "F.Cu")
@@
 	)
 	(segment
-		(start 114.8901 34.4338)
-		(end 116.2647 33.0592)
+		(start 116.2647 33.0592)
+		(end 116.2647 9.8387)
 		(width 0.2)
 		(layer "F.Cu")
@@
 	)
 	(segment
-		(start 116.2647 33.0592)
-		(end 116.2647 13.7127)
+		(start 110.8232 34.4338)
+		(end 114.8901 34.4338)
 		(width 0.2)
 		(layer "F.Cu")
@@
 	)
 	(segment
-		(start 35.6093 15.6987)
-		(end 31.75 19.558)
+		(start 90.174 22.098)
+		(end 89.0435 20.9675)
 		(width 0.2)
 		(layer "F.Cu")
@@
 	)
 	(segment
-		(start 89.879 13.208)
-		(end 92.9345 13.208)
+		(start 37.0285 5.7517)
+		(end 37.9416 6.6648)
 		(width 0.2)
 		(layer "F.Cu")
@@
 	)
 	(segment
-		(start 107.3868 8.9536)
-		(end 107.3868 6.8038)
+		(start 89.0435 20.9675)
+		(end 89.0435 14.0435)
 		(width 0.2)
 		(layer "F.Cu")
@@
 	)
 	(segment
-		(start 37.1312 13.208)
-		(end 36.5058 13.208)
+		(start 35.6093 14.1045)
+		(end 35.6093 15.6987)
 		(width 0.2)
 		(layer "F.Cu")
@@
 	)
 	(segment
-		(start 89.0435 20.9675)
-		(end 89.0435 14.0435)
+		(start 105.1355 2.7735)
+		(end 38.1247 2.7735)
 		(width 0.2)
 		(layer "F.Cu")
@@
 	)
 	(segment
-		(start 37.0285 5.7517)
-		(end 37.9416 6.6648)
+		(start 36.5058 13.208)
+		(end 35.6093 14.1045)
 		(width 0.2)
 		(layer "F.Cu")
@@
 	)
 	(segment
-		(start 37.9416 6.6648)
-		(end 37.9416 12.3976)
+		(start 89.0435 14.0435)
+		(end 89.879 13.208)
 		(width 0.2)
 		(layer "F.Cu")
@@
 	)
 	(segment
-		(start 103.3565 2.7735)
-		(end 38.1247 2.7735)
+		(start 95.6335 10.509)
+		(end 107.601 10.509)
 		(width 0.2)
 		(layer "F.Cu")
@@
 	)
 	(segment
-		(start 36.5058 13.208)
-		(end 35.6093 14.1045)
+		(start 107.601 10.509)
+		(end 109.035 9.075)
 		(width 0.2)
 		(layer "F.Cu")
@@
 	)
 	(segment
-		(start 95.6335 10.509)
-		(end 105.8314 10.509)
+		(start 37.9416 6.6648)
+		(end 37.9416 12.3976)
 		(width 0.2)
 		(layer "F.Cu")
@@
 	)
 	(segment
-		(start 38.1247 2.7735)
-		(end 37.0285 3.8697)
+		(start 89.879 13.208)
+		(end 92.9345 13.208)
 		(width 0.2)
 		(layer "F.Cu")
@@
 	)
 	(segment
-		(start 37.9416 12.3976)
-		(end 37.1312 13.208)
+		(start 92.9345 13.208)
+		(end 95.6335 10.509)
 		(width 0.2)
 		(layer "F.Cu")
@@
 	)
 	(segment
-		(start 90.174 22.098)
-		(end 89.0435 20.9675)
+		(start 37.0285 3.8697)
+		(end 37.0285 5.7517)
 		(width 0.2)
 		(layer "F.Cu")
@@
 	)
 	(segment
-		(start 37.0285 3.8697)
-		(end 37.0285 5.7517)
+		(start 109.035 9.075)
+		(end 109.035 6.673)
 		(width 0.2)
 		(layer "F.Cu")
@@
 	)
 	(segment
-		(start 107.3868 6.8038)
-		(end 103.3565 2.7735)
+		(start 38.1247 2.7735)
+		(end 37.0285 3.8697)
 		(width 0.2)
 		(layer "F.Cu")
@@
 	)
 	(segment
-		(start 105.8314 10.509)
-		(end 107.3868 8.9536)
+		(start 35.6093 15.6987)
+		(end 31.75 19.558)
 		(width 0.2)
 		(layer "F.Cu")
@@
 	)
 	(segment
-		(start 89.0435 14.0435)
-		(end 89.879 13.208)
+		(start 37.1312 13.208)
+		(end 36.5058 13.208)
 		(width 0.2)
 		(layer "F.Cu")
@@
 	)
 	(segment
-		(start 92.9345 13.208)
-		(end 95.6335 10.509)
+		(start 37.9416 12.3976)
+		(end 37.1312 13.208)
 		(width 0.2)
 		(layer "F.Cu")
@@
 	)
 	(segment
-		(start 35.6093 14.1045)
-		(end 35.6093 15.6987)
+		(start 109.035 6.673)
+		(end 105.1355 2.7735)
 		(width 0.2)
 		(layer "F.Cu")

Commit message: PCB updated
Parts:
- S1: value Button TACT 12x12mm -> Button TACT 6x6mm; footprint StockLib:Button TACT 12x12mm -> StockLib:Button TACT 6x6mm
- moved G1 108.3 mm to (113.0, 54.8), turned to -90 degrees
- moved C9 76.5 mm to (86.9, 51.8)
- moved C7 51.2 mm to (106.2, 6.10)
- moved U7 51.2 mm to (104.9, 11.2)
- moved D4 26.0 mm to (109.2, 33.8)
- moved C8 24.4 mm to (28.7, 49.5)
- moved J6 24.1 mm to (84.6, 32.5), turned to 0 degrees
- moved C6 23.7 mm to (93.5, 6.10)
- moved U6 23.7 mm to (92.2, 11.2)
- moved C10 23.3 mm to (71.6, 51.8)
- moved R6 21.9 mm to (92.2, 33.8)
- moved D3 21.9 mm to (92.3, 38.8)
- moved R3 21.9 mm to (92.3, 43.9)
- moved Y1 21.6 mm to (27.5, 41.1)
- moved R5 19.7 mm to (25.7, 54.6)
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Routing:
- net +5V: track 342.1 -> 0.00 mm
- net IO_~{M}: track 186.3 -> 0.00 mm
- net /D4: track 172.6 -> 0.00 mm
- net A15: track 171.6 -> 0.00 mm
- net /D5: track 145.6 -> 0.00 mm
- net RESET_OUT: track 145.5 -> 0.00 mm
- net Net-(D3-K): track 143.6 -> 0.00 mm
- net /D3: track 138.9 -> 0.00 mm
- net ~{RD}: track 137.8 -> 0.00 mm
- net UART_RX: track 134.6 -> 0.00 mm
- net /D6: track 133.8 -> 0.00 mm
- net UART_TX: track 130.7 -> 0.00 mm
- net /A8: track 127.5 -> 0.00 mm
- net Net-(U1-~{RESET_IN}): track 126.0 -> 0.00 mm
- net /A10: track 123.8 -> 0.00 mm
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
Commit message: PCB updated
Parts:
- added TP1: X1, TestPoint:TestPoint_THTPad_D1.0mm_Drill0.5mm, F.Cu at (37.6, 49.3)
- added TP10: ~{ROMEN}, TestPoint:TestPoint_THTPad_D1.0mm_Drill0.5mm, F.Cu at (89.7, 6.10)
- added TP2: X2, TestPoint:TestPoint_THTPad_D1.0mm_Drill0.5mm, F.Cu at (37.6, 54.4)
- added TP3: 5V, TestPoint:TestPoint_THTPad_D1.0mm_Drill0.5mm, F.Cu at (67.6, 51.3)
- added TP4: GND, TestPoint:TestPoint_THTPad_D1.0mm_Drill0.5mm, F.Cu at (67.6, 58.2)
- added TP5: IO/~{M}, TestPoint:TestPoint_THTPad_D1.0mm_Drill0.5mm, F.Cu at (21.8, 6.10)
- added TP6: ~{WR}, TestPoint:TestPoint_THTPad_D1.0mm_Drill0.5mm, F.Cu at (36.3, 6.10)
- added TP7: ~{RD}, TestPoint:TestPoint_THTPad_D1.0mm_Drill0.5mm, F.Cu at (40.1, 6.10)
- added TP8: RESET_OUT, TestPoint:TestPoint_THTPad_D1.0mm_Drill0.5mm, F.Cu at (56.6, 6.10)
- added TP9: ~{RAMEN}, TestPoint:TestPoint_THTPad_D1.0mm_Drill0.5mm, F.Cu at (74.9, 5.84)
- J1: footprint Connector_Dsub:DSUB-9_Pins_Horizontal_P2.77x2.84mm_EdgePinOffset9.90mm_Housed_MountingHolesOffset11.32mm -> Connector_Dsub:DSUB-9_Socket_Horizontal_P2.77x2.84mm_EdgePinOffset9.90mm_Housed_MountingHolesOffset11.32mm
- moved R4 15.3 mm to (35.1, 44.2)
- moved R5 15.3 mm to (24.9, 39.4)
- moved J1 11.1 mm to (56.8, 66.9)
- moved Y1 10.2 mm to (27.3, 51.3)
- moved C8 9.91 mm to (28.5, 59.4)
- moved J2 0.19 mm to (25.4, 68.9)
Routing:
- net +5V: track 0.00 -> 391.2 mm
- net A15: track 0.00 -> 245.3 mm
- net Net-(U1-~{RESET_IN}): track 0.00 -> 238.6 mm
- net ~{RD}: track 0.00 -> 189.6 mm
- net RESET_OUT: track 0.00 -> 187.4 mm
- net UART_TX: track 0.00 -> 164.6 mm
- net ~{WR}: track 0.00 -> 162.5 mm
- net UART_RX: track 0.00 -> 155.1 mm
- net /A8: track 0.00 -> 154.4 mm
- net /D6: track 0.00 -> 139.9 mm
- net /D5: track 0.00 -> 135.6 mm
- net IO_~{M}: track 0.00 -> 108.9 mm
- net /D4: track 0.00 -> 108.6 mm
- net /A9: track 0.00 -> 108.3 mm
- net /D3: track 0.00 -> 104.7 mm
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Other:
- board text added: "8085 EXPLORER SINGLE BOARD COMPUTER V1.0"
- board text added: "IO/~{M}"
- board text added: "RESET_OUT"
- board text added: "X1"
- board text added: "X2"
- board text added: "~{RAMEN}"
- board text added: "~{RD}"
- board text added: "~{ROMEN}"
- board text added: "~{WR}"
- board text removed: "NETRONICS EXPLORER/85 SINGLE BOARD COMPUTER V1.0"

Commit message: PCB updated
Parts:
- R1, R2, R6: value 470R -> 1k; footprint StockLib:R_470_Axial_DIN0207 -> StockLib:R_1k_Axial_DIN0207
Changed lines of the file:
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@@
 		)
 	)
-	(footprint "StockLib:R_470_Axial_DIN0207"
+	(footprint "StockLib:R_1k_Axial_DIN0207"
 		(layer "F.Cu")
 		(at 96.012 64.516)
@@
 			)
 		)
-		(property "Value" "470R"
+		(property "Value" "1k"
 			(at 5.08 2.37 0)
 			(layer "F.Fab")
@@
 		)
 		(embedded_fonts no)
-		(model "${KICAD_USER_3DMODEL_DIR}/Resistors/Res-10.16-6.3x2.3-470.step"
+		(model "${KICAD_USER_3DMODEL_DIR}/Resistors/Res-10.16-6.3x2.3-1k.step"
 			(offset
 				(xyz 5 0 0)
@@
 		)
 	)
-	(footprint "StockLib:R_470_Axial_DIN0207"
+	(footprint "StockLib:R_1k_Axial_DIN0207"
 		(layer "F.Cu")
 		(at 92.202 33.782)
@@
 			)
 		)
-		(property "Value" "470R"
+		(property "Value" "1k"
 			(at 5.08 2.37 0)
 			(layer "F.Fab")
@@
 		)
 		(embedded_fonts no)
-		(model "${KICAD_USER_3DMODEL_DIR}/Resistors/Res-10.16-6.3x2.3-470.step"
+		(model "${KICAD_USER_3DMODEL_DIR}/Resistors/Res-10.16-6.3x2.3-1k.step"
 			(offset
 				(xyz 5 0 0)
@@
 		)
 	)
-	(footprint "StockLib:R_470_Axial_DIN0207"
+	(footprint "StockLib:R_1k_Axial_DIN0207"
 		(layer "F.Cu")
 		(at 96.012 59.69)
@@
 			)
 		)
-		(property "Value" "470R"
+		(property "Value" "1k"
 			(at 5.08 2.37 0)
 			(layer "F.Fab")
@@
 		)
 		(embedded_fonts no)
-		(model "${KICAD_USER_3DMODEL_DIR}/Resistors/Res-10.16-6.3x2.3-470.step"
+		(model "${KICAD_USER_3DMODEL_DIR}/Resistors/Res-10.16-6.3x2.3-1k.step"
 			(offset
 				(xyz 5 0 0)
@@
 	)
 	(gr_text "TX"
-		(at 101.6 72.898 90)
+		(at 102.362 72.898 90)
 		(layer "F.SilkS")
 		(effects
@@
 	)
 	(gr_text "RX"
-		(at 93.467 72.898 90)
+		(at 94.234 72.898 90)
 		(layer "F.SilkS")
 		(effects
