File: schematic/8085-explorer.kicad_sch (KiCad schematic)
At the start: 43 parts, among them J1 DE9_Pins_MountingHoles, J2 DC-005 Power Jack, U1 8085, U2 74LS573, U3 L7805, U4 28C256, U5 74LS14, U6 74LS32, U7 74LS74, U8 HM62256BLP, U9 MAX232, Y1 6.144 MHz

Commit message: PCB updated
Parts:
- added J4, J5: Conn_01x02_Pin, Connector_PinHeader_2.54mm:PinHeader_1x02_P2.54mm_Vertical, symbol Connector:Conn_01x02_Pin
- added J6: Conn_02x05_Odd_Even, Connector_PinSocket_2.54mm:PinSocket_2x05_P2.54mm_Vertical, symbol Connector_Generic:Conn_02x05_Odd_Even
- renumbered C2 to C1, C13 to C10, C17 to C11, C14 to C12, C16 to C13, C15 to C14, C1 to C15, C10 to C16, C10 to C17, C12 to C18, C3 to C2, C4 to C3, C5 to C4, C6 to C5, C8 to C6, C9 to C7, C11 to C8, C7 to C9, D3 to D1, D5 to D3, D6 to D4, D1 to D5, R2 to R1, R5 to R2, R1 to R3, R3 to R4, R4 to R5, R11 to R6, U4 to U3, U8 to U4, U9 to U8, U3 to U9
Connections:
- net +5V: now also J6.1 (Pin_1), J6.3 (Pin_3), J6.5 (Pin_5), J6.7 (Pin_7), J6.9 (Pin_9)
- net GND: now also J6.10 (Pin_10), J6.2 (Pin_2), J6.4 (Pin_4), J6.6 (Pin_6), J6.8 (Pin_8)
- net UART_RX: now also J5.1 (Pin_1); no longer U8.12 (R1OUT)
- net UART_TX: now also J4.1 (Pin_1); no longer U8.11 (T1IN)
- new net: J5.2 (Pin_2), U8.12 (R1OUT)
- new net: J4.2 (Pin_2), U8.11 (T1IN)
- no-connect marks 21 -> 22
Other:
- moved on the sheet: C10, C11, C12, C13, C14, D4, J1, J2, R6, U5A, U5F, U7A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

Commit message: PCB updated
Other:
- note added: "Glue logic"
- note added: "Microprocessor system"
- note added: "Power"
- note added: "Serial output"
- moved on the sheet: C1, C10, C11, C12, C13, C14, C15, C16, C17, C18, C2, C3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

Commit message: PCB updated
Parts:
- removed S1: Button TACT 12x12mm, StockLib:Button TACT 12x12mm, symbol StockLib:Button TACT 12x12mm
- added S1: Button TACT 6x6mm, StockLib:Button TACT 6x6mm, symbol StockLib:Button TACT 6x6mm
Connections:
- net GND: now also S1.2
- net at C9.1, D3.1 (K), R3.1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: now also S1.3
Changed lines of the file:
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@@
+	)
+	(symbol
+		(lib_id "StockLib:Button TACT 6x6mm")
+		(at 177.8 151.13 0)
+		(unit 1)
+		(exclude_from_sim no)
+		(in_bom yes)
+		(on_board yes)
+		(dnp no)
+		(fields_autoplaced yes)
+		(property "Reference" "S1"
+			(at 177.8 138.43 0)
+			(effects
+				(font
+					(size 1.27 1.27)
+				)
+			)
+		)
+		(property "Value" "Button TACT 6x6mm"
+			(at 177.8 140.97 0)
+			(effects
+				(font
+					(size 1.27 1.27)
+				)
+			)
+		)
+		(property "Footprint" "StockLib:Button TACT 6x6mm"
+			(at 177.8 151.13 0)
+			(effects
+				(font
+					(size 1.27 1.27)
+				)
+				(justify bottom)
+				(hide yes)
+			)
+		)
+		(property "Datasheet" ""
+			(at 177.8 151.13 0)
+			(effects
+				(font
+					(size 1.27 1.27)
+				)
+				(hide yes)
+			)
+		)
+		(property "Description" "6 x 6 mm, 10 mm Actuator Height, 260 gf, Black, Long Crimped, Through Hole, SPST, Tactile Switch"
+			(at 177.8 151.13 0)
+			(effects
+				(font
+					(size 1.27 1.27)
+				)
+				(justify bottom)
+				(hide yes)
+			)
+		)
+		(property "MF" "CUI Devices"
+			(at 177.8 151.13 0)
+			(effects
+				(font
+					(size 1.27 1.27)
+				)
+				(justify bottom)
+				(hide yes)
+			)
+		)
+		(property "Package" "None"
+			(at 177.8 151.13 0)
+			(effects
+				(font
+					(size 1.27 1.27)
+				)
+				(justify bottom)
+				(hide yes)
+			)
+		)
+		(property "Price" "None"
+			(at 177.8 151.13 0)
+			(effects
+				(font
+					(size 1.27 1.27)
+				)
+				(justify bottom)
+				(hide yes)
+			)
+		)
+		(property "Check_prices" "https://www.snapeda.com/parts/TS02-66-100-BK-260-LCR-D/CUI+Devices/view-part/?ref=eda"
+			(at 177.8 151.13 0)
+			(effects
+				(font
+					(size 1.27 1.27)
+				)
+				(justify bottom)
+				(hide yes)
+			)
+		)
+		(property "STANDARD" "Manufacturer Recommendations"
+			(at 177.8 151.13 0)
+			(effects
+				(font
+					(size 1.27 1.27)
+				)
+				(justify bottom)
+				(hide yes)
+			)
+		)
+		(property "PARTREV" "1.0"
+			(at 177.8 151.13 0)
+			(effects
+				(font
+					(size 1.27 1.27)
+				)
+				(justify bottom)
+				(hide yes)
+			)
+		)
+		(property "SnapEDA_Link" "https://www.snapeda.com/parts/TS02-66-100-BK-260-LCR-D/CUI+Devices/view-part/?ref=snap"
+			(at 177.8 151.13 0)
+			(effects
+				(font
+					(size 1.27 1.27)
+				)
+				(justify bottom)
+				(hide yes)
+			)
+		)
+		(property "MP" "TS02-66-100-BK-260-LCR-D"
+			(at 177.8 151.13 0)
+			(effects
+				(font
+					(size 1.27 1.27)
+				)
+				(justify bottom)
+				(hide yes)
+			)
+		)
+		(property "CUI_purchase_URL" "https://www.cuidevices.com/product/switches/tactile-switches/ts02-66-100-bk-260-lcr-d?utm_source=snapeda.com&utm_medium=referral&utm_campaign=snapedaBOM"
+			(at 177.8 151.13 0)
+			(effects
+				(font
+					(size 1.27 1.27)
+				)
+				(justify bottom)
+				(hide yes)
+			)
+		)
+		(property "Availability" "In Stock"
+			(at 177.8 151.13 0)
+			(effects
+				(font
+					(size 1.27 1.27)
+				)
+				(justify bottom)
+				(hide yes)
+			)
+		)
+		(property "MANUFACTURER" "CUI Devices"
+			(at 177.8 151.13 0)
+			(effects
+				(font
+					(size 1.27 1.27)
+				)
+				(justify bottom)
+				(hide yes)
+			)
+		)
+		(pin "2"
+		)
+		(pin "3"
+		)
+		(pin "1"
+		)
+		(pin "4"
+		)
+		(instances
+			(project ""
+				(path "/ddfadebd-517c-41ab-bf2b-16caab502112"
+					(reference "S1")
+					(unit 1)
+				)
+			)
+		)
 	)
 	(symbol
@@
 					(unit 1)
 				)
-			)
-		)
-	)
-	(symbol
-		(lib_id "StockLib:Button TACT 12x12mm")
-		(at 177.8 151.13 0)
-		(unit 1)
-		(exclude_from_sim no)
-		(in_bom yes)
-		(on_board yes)
-		(dnp no)
-		(fields_autoplaced yes)
-		(property "Reference" "S1"
-			(at 177.8 138.43 0)
-			(effects
-				(font
-					(size 1.27 1.27)
-				)
-			)
-		)
-		(property "Value" "Button TACT 12x12mm"
-			(at 177.8 140.97 0)
-			(effects
-				(font
-					(size 1.27 1.27)
-				)
-			)
-		)
-		(property "Footprint" "StockLib:Button TACT 12x12mm"
-			(at 177.8 151.13 0)
-			(effects
-				(font
-					(size 1.27 1.27)
-				)
-				(justify bottom)
-				(hide yes)
-			)
-		)
-		(property "Datasheet" ""
-			(at 177.8 151.13 0)
-			(effects
-				(font
-					(size 1.27 1.27)
-				)
-				(hide yes)
-			)
-		)
-		(property "Description" "12 x 12 mm, 10 mm Actuator Height, 260 gf, Black, Long Crimped, Through Hole, SPST, Tactile Switch"
-			(at 177.8 151.13 0)
-			(effects
-				(font
-					(size 1.27 1.27)
-				)
-				(justify bottom)
-				(hide yes)
-			)
-		)
-		(property "MF" "CUI Devices"
-			(at 177.8 151.13 0)
-			(effects
-				(font
-					(size 1.27 1.27)
-				)
-				(justify bottom)
-				(hide yes)
-			)
-		)
-		(property "Package" "None"
-			(at 177.8 151.13 0)
-			(effects
-				(font
-					(size 1.27 1.27)
-				)
-				(justify bottom)
-				(hide yes)
-			)
-		)
-		(property "Price" "None"
-			(at 177.8 151.13 0)
-			(effects
-				(font
-					(size 1.27 1.27)
-				)
-				(justify bottom)
-				(hide yes)
-			)
-		)
-		(property "Check_prices" "https://www.snapeda.com/parts/TS02-66-100-BK-260-LCR-D/CUI+Devices/view-part/?ref=eda"
-			(at 177.8 151.13 0)
-			(effects
-				(font
-					(size 1.27 1.27)
-				)
-				(justify bottom)
-				(hide yes)
-			)
-		)
-		(property "STANDARD" "Manufacturer Recommendations"
-			(at 177.8 151.13 0)
-			(effects
-				(font
-					(size 1.27 1.27)
-				)
-				(justify bottom)
-				(hide yes)
-			)
-		)
-		(property "PARTREV" "1.0"
-			(at 177.8 151.13 0)
-			(effects
-				(font
-					(size 1.27 1.27)
-				)
-				(justify bottom)
-				(hide yes)
-			)
-		)
-		(property "SnapEDA_Link" "https://www.snapeda.com/parts/TS02-66-100-BK-260-LCR-D/CUI+Devices/view-part/?ref=snap"
-			(at 177.8 151.13 0)
-			(effects
-				(font
-					(size 1.27 1.27)
-				)
-				(justify bottom)
-				(hide yes)
-			)
-		)
-		(property "MP" "TS02-66-100-BK-260-LCR-D"
-			(at 177.8 151.13 0)
-			(effects
-				(font
-					(size 1.27 1.27)
-				)
-				(justify bottom)
-				(hide yes)
-			)
-		)
-		(property "CUI_purchase_URL" "https://www.cuidevices.com/product/switches/tactile-switches/ts02-66-100-bk-260-lcr-d?utm_source=snapeda.com&utm_medium=referral&utm_campaign=snapedaBOM"
-			(at 177.8 151.13 0)
-			(effects
-				(font
-					(size 1.27 1.27)
-				)
-				(justify bottom)
-				(hide yes)
-			)
-		)
-		(property "Availability" "In Stock"
-			(at 177.8 151.13 0)
-			(effects
-				(font
-					(size 1.27 1.27)
-				)
-				(justify bottom)
-				(hide yes)
-			)
-		)
-		(property "MANUFACTURER" "CUI Devices"
-			(at 177.8 151.13 0)
-			(effects
-				(font
-					(size 1.27 1.27)
-				)
-				(justify bottom)
-				(hide yes)
-			)
-		)
-		(pin "1"
-		)
-		(pin "2"
-		)
-		(pin "4"
-		)
-		(pin "3"
-		)
-		(instances
-			(project ""
-				(path "/ddfadebd-517c-41ab-bf2b-16caab502112"
-					(reference "S1")
-					(unit 1)
-				)

Commit message: PCB updated
Parts:
- added TP1: X1, TestPoint:TestPoint_THTPad_D1.0mm_Drill0.5mm, symbol Connector:TestPoint
- added TP10: ~{ROMEN}, TestPoint:TestPoint_THTPad_D1.0mm_Drill0.5mm, symbol Connector:TestPoint
- added TP2: X2, TestPoint:TestPoint_THTPad_D1.0mm_Drill0.5mm, symbol Connector:TestPoint
- added TP3: 5V, TestPoint:TestPoint_THTPad_D1.0mm_Drill0.5mm, symbol Connector:TestPoint
- added TP4: GND, TestPoint:TestPoint_THTPad_D1.0mm_Drill0.5mm, symbol Connector:TestPoint
- added TP5: IO/~{M}, TestPoint:TestPoint_THTPad_D1.0mm_Drill0.5mm, symbol Connector:TestPoint
- added TP6: ~{WR}, TestPoint:TestPoint_THTPad_D1.0mm_Drill0.5mm, symbol Connector:TestPoint
- added TP7: ~{RD}, TestPoint:TestPoint_THTPad_D1.0mm_Drill0.5mm, symbol Connector:TestPoint
- added TP8: RESET_OUT, TestPoint:TestPoint_THTPad_D1.0mm_Drill0.5mm, symbol Connector:TestPoint
- added TP9: ~{RAMEN}, TestPoint:TestPoint_THTPad_D1.0mm_Drill0.5mm, symbol Connector:TestPoint
- J1: footprint Connector_Dsub:DSUB-9_Pins_Horizontal_P2.77x2.84mm_EdgePinOffset9.90mm_Housed_MountingHolesOffset11.32mm -> Connector_Dsub:DSUB-9_Socket_Horizontal_P2.77x2.84mm_EdgePinOffset9.90mm_Housed_MountingHolesOffset11.32mm
Connections:
- net +5V: now also TP3.1
- net GND: now also TP4.1
- net IO_~{M}: now also TP5.1
- net RESET_OUT: now also TP8.1
- net ~{RAMEN}: now also TP9.1
- net ~{RD}: now also TP7.1
- net ~{ROMEN}: now also TP10.1
- net ~{WR}: now also TP6.1
- net at C8.1, U1.2 (X2), Y1.1: now also TP2.1
- net at U1.1 (X1), Y1.2: now also TP1.1
Other:
- moved on the sheet: C8, Y1

Commit message: PCB updated
Parts:
- R1, R2, R6: value 470R -> 1k; footprint StockLib:R_470_Axial_DIN0207 -> StockLib:R_1k_Axial_DIN0207
Changed lines of the file:
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@@
 		(fields_autoplaced yes)
 		(property "Reference" "R6"
-			(at 36.83 254 90)
+			(at 33.02 252.7299 0)
 			(effects
 				(font
 					(size 1.27 1.27)
 				)
+				(justify left)
 			)
 		)
-		(property "Value" "470R"
-			(at 34.29 254 90)
+		(property "Value" "1k"
+			(at 33.02 255.2699 0)
 			(effects
 				(font
 					(size 1.27 1.27)
 				)
+				(justify left)
 			)
 		)
-		(property "Footprint" "StockLib:R_470_Axial_DIN0207"
+		(property "Footprint" "StockLib:R_1k_Axial_DIN0207"
 			(at 28.702 254 90)
 			(effects
@@
 		(fields_autoplaced yes)
 		(property "Reference" "R2"
-			(at 132.08 120.65 90)
+			(at 128.27 119.3799 0)
 			(effects
 				(font
 					(size 1.27 1.27)
 				)
+				(justify left)
 			)
 		)
-		(property "Value" "470R"
-			(at 129.54 120.65 90)
+		(property "Value" "1k"
+			(at 128.27 121.9199 0)
 			(effects
 				(font
 					(size 1.27 1.27)
 				)
+				(justify left)
 			)
 		)
-		(property "Footprint" "StockLib:R_470_Axial_DIN0207"
+		(property "Footprint" "StockLib:R_1k_Axial_DIN0207"
 			(at 123.952 120.65 90)
 			(effects
@@
 		(fields_autoplaced yes)
 		(property "Reference" "R1"
-			(at 119.38 120.65 90)
+			(at 115.57 119.3799 0)
 			(effects
 				(font
 					(size 1.27 1.27)
 				)
+				(justify left)
 			)
 		)
-		(property "Value" "470R"
-			(at 116.84 120.65 90)
+		(property "Value" "1k"
+			(at 115.57 121.9199 0)
 			(effects
 				(font
 					(size 1.27 1.27)
 				)
+				(justify left)
 			)
 		)
-		(property "Footprint" "StockLib:R_470_Axial_DIN0207"
+		(property "Footprint" "StockLib:R_1k_Axial_DIN0207"
 			(at 111.252 120.65 90)
 			(effects
